Commit message: ok ok its good

File: src/robot_simulation/urdf/robot.urdf.xacro (robot description, xacro)
@@ -24,5 +24,5 @@
     <xacro:property name="caster_width"  value="0.03"/>
     <xacro:property name="caster_x" value="0.18"/>
-    <xacro:property name="caster_z" value="-0.06"/>
+    <xacro:property name="caster_z" value="-0.1"/>
     <!-- ================================================== -->
     <!-- CHÂSSIS                                           -->
@@ -190,5 +190,5 @@
         <parent link="base_link"/>
         <child link="lidar_link"/>
-        <origin xyz="0.22 0 0.066" rpy="0 0 0"/>
+        <origin xyz="0.25 0 0.066" rpy="0 0 0"/>
     </joint>
     <!-- ================================================== -->
@@ -197,5 +197,5 @@
     <gazebo reference="lidar_link">
         <sensor name="front_lidar" type="gpu_lidar">
-            <topic>/simulation/distance</topic>
+            <topic>/simulation/lidar_points</topic>
             <update_rate>10</update_rate>
             <always_on>true</always_on>
@@ -210,12 +210,12 @@
                     </horizontal>
                     <vertical>
-                        <samples>1</samples>
+                        <samples>3</samples>
                         <resolution>1</resolution>
-                        <min_angle>0.1</min_angle>
-                        <max_angle>0.1</max_angle>
+                        <min_angle>-1.0472</min_angle>
+                        <max_angle>0.0</max_angle>
                     </vertical>
                 </scan>
                 <range>
-                    <min>0.5</min>
+                    <min>0.05</min>
                     <max>15.0</max>
                     <resolution>0.01</resolution>
@@ -224,3 +224,13 @@
         </sensor>
     </gazebo>
+    <gazebo>
+        <plugin filename="gz-sim-diff-drive-system" name="gz::sim::systems::DiffDrive">
+            <left_joint>left_wheel_joint</left_joint>
+            <right_joint>right_wheel_joint</right_joint>
+            <wheel_separation>0.33</wheel_separation>
+            <wheel_radius>0.05</wheel_radius>
+            <topic>/cmd_vel</topic>
+            <odom_publish_frequency>30</odom_publish_frequency>
+        </plugin>
+    </gazebo>
 </robot>

Commit message: Refactoring all system

File: src/robot_simulation/urdf/robot.urdf.xacro (robot description, xacro)
@@ -2,32 +2,26 @@
 <robot xmlns:xacro="http://www.ros.org/wiki/xacro" name="robot">
     <!-- ================================================== -->
-    <!-- Dimensions générales du robot                     -->
-    <!-- ================================================== -->
+    <!-- PROPRIÉTÉS GÉNÉRALES                               -->
+    <!-- ================================================== -->
+    <!-- Châssis -->
     <xacro:property name="base_length" value="0.40"/>
     <xacro:property name="base_width"  value="0.30"/>
     <xacro:property name="base_height" value="0.12"/>
-    <!-- Position du centre du châssis -->
-    <xacro:property name="base_z" value="0.11"/>
-    <!-- ================================================== -->
-    <!-- Roues arrière                                     -->
-    <!-- ================================================== -->
-    <xacro:property name="wheel_radius" value="0.05"/>
-    <xacro:property name="wheel_width"  value="0.03"/>
-    <!-- Position des roues -->
-    <xacro:property name="wheel_x" value="-0.10"/>
-    <xacro:property name="wheel_y" value="0.165"/>
-    <xacro:property name="wheel_z" value="-0.08"/>
-    <!-- ================================================== -->
-    <!-- Roue directrice avant                             -->
-    <!-- ================================================== -->
-    <xacro:property name="caster_radius" value="0.04"/>
-    <xacro:property name="caster_width"  value="0.03"/>
-    <xacro:property name="caster_x" value="0.18"/>
-    <xacro:property name="caster_z" value="-0.1"/>
-    <!-- ================================================== -->
-    <!-- CHÂSSIS                                           -->
+    <!-- Roues motrices -->
+    <xacro:property name="wheel_radius" value="0.15"/>
+    <xacro:property name="wheel_width"  value="0.06"/>
+    <!-- Position des roues motrices              -->
+    <!-- Les roues sont légèrement vers l'arrière -->
+    <xacro:property name="wheel_x" value="-0.08"/>
+    <xacro:property name="wheel_y" value="0.18"/>
+    <xacro:property name="wheel_z" value="0.0"/>
+    <!-- Caster -->
+    <xacro:property name="caster_x" value="0.13"/>
+    <xacro:property name="caster_radius" value="0.06"/>
+    <xacro:property name="caster_width" value="0.04"/>
+    <!-- ================================================== -->
+    <!-- CHÂSSIS                                            -->
     <!-- ================================================== -->
     <link name="base_link">
-        <!-- Visualisation -->
         <visual>
             <origin xyz="0 0 0"/>
@@ -39,40 +33,38 @@
             </material>
         </visual>
-        <!-- Collision -->
-        <collision>
-            <origin xyz="0 0 0"/>
-            <geometry>
-                <box size="${base_length} ${base_width} ${base_height}"/>
-            </geometry>
-        </collision>
-        <!-- Physique -->
+        <collision>
+            <origin xyz="0 0 0"/>
+            <geometry>
+                <box size="${base_length} ${base_width} ${base_height}" />
+            </geometry>
+        </collision>
         <inertial>
             <origin xyz="0 0 0"/>
             <mass value="5.0"/>
             <inertia
-                ixx="0.045"
-                ixy="0.0"
-                ixz="0.0"
-                iyy="0.071"
-                iyz="0.0"
-                izz="0.092"/>
-        </inertial>
-    </link>
-    <!-- ================================================== -->
-    <!-- ROUE ARRIÈRE GAUCHE                               -->
+                ixx="0.0453"
+                ixy="0.0"
+                ixz="0.0"
+                iyy="0.0713"
+                iyz="0.0"
+                izz="0.1042"
+            />
+        </inertial>
+    </link>
+    <!-- ================================================== -->
+    <!-- ROUE MOTRICE GAUCHE                                -->
     <!-- ================================================== -->
     <link name="left_wheel">
         <visual>
-            <!-- Le cylindre tourne autour de Y -->
-            <origin xyz="0 0 0" rpy="1.5708 0 0"/>
-            <geometry>
-                <cylinder radius="${wheel_radius}" length="${wheel_width}" />
-            </geometry>
-            <material name="left_wheel_color">
+            <origin xyz="0 0 0" rpy="1.5708 0 0" />
+            <geometry>
+                <cylinder radius="${wheel_radius}" length="${wheel_width}" />
+            </geometry>
+            <material name="wheel_color">
                 <color rgba="0.6 0.0 1.0 1.0"/>
             </material>
         </visual>
         <collision>
-            <origin xyz="0 0 0" rpy="1.5708 0 0"/>
+            <origin xyz="0 0 0" rpy="1.5708 0 0" />
             <geometry>
                 <cylinder radius="${wheel_radius}" length="${wheel_width}" />
@@ -83,36 +75,41 @@
             <mass value="0.5"/>
             <inertia
-                ixx="0.0008"
-                ixy="0.0"
-                ixz="0.0"
-                iyy="0.0008"
-                iyz="0.0"
-                izz="0.0008"/>
-        </inertial>
-    </link>
+                ixx="0.00945"
+                ixy="0.0"
+                ixz="0.0"
+                iyy="0.005625"
+                iyz="0.0"
+                izz="0.00945"
+            />
+        </inertial>
+    </link>
+    <!-- Joint roue gauche -->
     <joint name="left_wheel_joint" type="continuous">
         <parent link="base_link"/>
         <child link="left_wheel"/>
-        <origin xyz="${wheel_x} ${wheel_y} ${wheel_z}" rpy="0 0 0"/>
+        <origin
+            xyz="${wheel_x} ${wheel_y} ${wheel_z}"
+            rpy="0 0 0"
+        />
         <!-- Axe de rotation de la roue -->
         <axis xyz="0 1 0"/>
     </joint>
-    <!-- ================================================== -->
-    <!-- ROUE ARRIÈRE DROITE                               -->
-    <!-- ================================================== -->
+<!-- ================================================== -->
+<!-- ROUE MOTRICE DROITE                                -->
+<!-- ================================================== -->
     <link name="right_wheel">
         <visual>
-            <origin xyz="0 0 0" rpy="1.5708 0 0"/>
-            <geometry>
-                <cylinder radius="${wheel_radius}" length="${wheel_width}" />
-            </geometry>
-            <material name="right_wheel_color">
+            <origin xyz="0 0 0" rpy="1.5708 0 0" />
+            <geometry>
+                <cylinder radius="${wheel_radius}" length="${wheel_width}" />
+            </geometry>
+            <material name="wheel_color">
                 <color rgba="0.6 0.0 1.0 1.0"/>
             </material>
         </visual>
         <collision>
-            <origin xyz="0 0 0" rpy="1.5708 0 0"/>
-            <geometry>
-                <cylinder radius="${wheel_radius}" length="${wheel_width}"/>
+            <origin xyz="0 0 0" rpy="1.5708 0 0" />
+            <geometry>
+                <cylinder radius="${wheel_radius}" length="${wheel_width}" />
             </geometry>
         </collision>
@@ -121,35 +118,79 @@
             <mass value="0.5"/>
             <inertia
-                ixx="0.0008"
-                ixy="0.0"
-                ixz="0.0"
-                iyy="0.0008"
-                iyz="0.0"
-                izz="0.0008"/>
-        </inertial>
-    </link>
+                ixx="0.00945"
+                ixy="0.0"
+                ixz="0.0"
+                iyy="0.005625"
+                iyz="0.0"
+                izz="0.00945"
+            />
+        </inertial>
+    </link>
+    <!-- Joint roue droite -->
     <joint name="right_wheel_joint" type="continuous">
         <parent link="base_link"/>
         <child link="right_wheel"/>
-        <origin xyz="${wheel_x} ${-wheel_y} ${wheel_z}" rpy="0 0 0"/>
+        <origin xyz="${wheel_x} ${-wheel_y} ${wheel_z}" rpy="0 0 0" />
+        <!-- Axe de rotation de la roue -->
         <axis xyz="0 1 0"/>
     </joint>
     <!-- ================================================== -->
-    <!-- ROUE DIRECTRICE AVANT                             -->
-    <!-- ================================================== -->
-    <link name="front_caster">
-        <visual>
-            <origin xyz="0 0 0" rpy="1.5708 0 0"/>
+    <!-- SUPPORT DU CASTER                                  -->
+    <!-- ================================================== -->
+    <link name="caster_fork">
+        <visual>
+            <origin xyz="0 0 0"/>
+            <geometry>
+                <cylinder radius="0.025" length="0.08" />
+            </geometry>
+            <material name="caster_fork_color">
+                <color rgba="0.15 0.15 0.15 1.0"/>
+            </material>
+        </visual>
+        <collision>
+            <origin xyz="0 0 0"/>
+            <geometry>
+                <cylinder radius="0.025" length="0.08" />
+            </geometry>
+        </collision>
+        <inertial>
+            <origin xyz="0 0 0"/>
+            <mass value="0.15"/>
+            <inertia
+                ixx="0.0001"
+                ixy="0.0"
+                ixz="0.0"
+                iyy="0.0001"
+                iyz="0.0"
+                izz="0.0001"
+            />
+        </inertial>
+    </link>
+    <!-- Axe vertical permettant au caster de s'orienter -->
+    <joint name="caster_swivel_joint" type="continuous">
+        <parent link="base_link"/>
+        <child link="caster_fork"/>
+        <origin xyz="${caster_x} 0 -0.06" rpy="0 0 0" />
+        <!-- Rotation du caster autour de Z -->
+        <axis xyz="0 0 1"/>
+    </joint>
+    <!-- ================================================== -->
+    <!-- ROUE DU CASTER                                     -->
+    <!-- ================================================== -->
+    <link name="caster_wheel">
+        <visual>
+            <!-- Roue dont l'axe est Y -->
+            <origin xyz="0 0 0" rpy="1.5708 0 0" />
             <geometry>
                 <cylinder radius="${caster_radius}" length="${caster_width}" />
             </geometry>
-            <material name="front_caster_color">
-                <color rgba="0.2 1.0 0.0 1.0"/>
-            </material>
-        </visual>
-        <collision>
-            <origin xyz="0 0 0" rpy="1.5708 0 0"/>
-            <geometry>
-                <cylinder radius="${caster_radius}" length="${caster_width}"/>
+            <material name="caster_wheel_color">
+                <color rgba="0.25 0.25 0.25 1.0"/>
+            </material>
+        </visual>
+        <collision>
+            <origin xyz="0 0 0" rpy="1.5708 0 0" />
+            <geometry>
+                <cylinder radius="${caster_radius}" length="${caster_width}" />
             </geometry>
         </collision>
@@ -158,21 +199,23 @@
             <mass value="0.2"/>
             <inertia
-                ixx="0.0003"
-                ixy="0.0"
-                ixz="0.0"
-                iyy="0.0003"
-                iyz="0.0"
-                izz="0.0003"/>
-        </inertial>
-    </link>
-    <joint name="front_caster_joint" type="continuous">
-        <parent link="base_link"/>
-        <child link="front_caster"/>
-        <origin xyz="${caster_x} 0 ${caster_z}" rpy="0 0 0"/>
-        <!-- Pour l'instant, roue libre -->
-        <axis xyz="0 0 1"/>
-    </joint>
-    <!-- ================================================== -->
-    <!-- CAPTEUR DE DISTANCE                               -->
+                ixx="0.0005"
+                ixy="0.0"
+                ixz="0.0"
+                iyy="0.00036"
+                iyz="0.0"
+                izz="0.0005"
+            />
+        </inertial>
+    </link>
+    <!-- Rotation de la roue du caster -->
+    <joint name="caster_wheel_joint" type="continuous">
+        <parent link="caster_fork"/>
+        <child link="caster_wheel"/>
+        <origin xyz="0 0 -0.06" rpy="0 0 0" />
+        <!-- Axe de rotation de la roue -->
+        <axis xyz="0 1 0"/>
+    </joint>
+    <!-- ================================================== -->
+    <!-- LiDAR                                              -->
     <!-- ================================================== -->
     <link name="lidar_link">
@@ -180,5 +223,5 @@
             <origin xyz="0 0 0"/>
             <geometry>
-                <cylinder radius="0.025" length="0.02"/>
+                <cylinder radius="0.025" length="0.02" />
             </geometry>
             <material name="lidar_color">
@@ -186,12 +229,25 @@
             </material>
         </visual>
-    </link>
+        <inertial>
+            <origin xyz="0 0 0"/>
+            <mass value="0.1"/>
+            <inertia
+                ixx="0.00001"
+                ixy="0.0"
+                ixz="0.0"
+                iyy="0.00001"
+                iyz="0.0"
+                izz="0.00001"
+            />
+        </inertial>
+    </link>
+    <!-- Position du LiDAR -->
     <joint name="lidar_joint" type="fixed">
         <parent link="base_link"/>
         <child link="lidar_link"/>
-        <origin xyz="0.25 0 0.066" rpy="0 0 0"/>
-    </joint>
-    <!-- ================================================== -->
-    <!-- CAPTEUR GAZEBO                                    -->
+        <origin xyz="0.25 0 0.066" rpy="0 0 0" />
+    </joint>
+    <!-- ================================================== -->
+    <!-- CAPTEUR LiDAR GAZEBO                               -->
     <!-- ================================================== -->
     <gazebo reference="lidar_link">
@@ -203,17 +259,20 @@
             <lidar>
                 <scan>
+                    <!-- Balayage horizontal -->
                     <horizontal>
-                        <samples>3</samples>
+                        <samples>360</samples>
                         <resolution>1</resolution>
-                        <min_angle>-0.5</min_angle>
-                        <max_angle>0.5</max_angle>
+                        <min_angle>-1.5708</min_angle>
+                        <max_angle>1.5708</max_angle>
                     </horizontal>
+                    <!-- Balayage vertical -->
                     <vertical>
-                        <samples>3</samples>
+                        <samples>16</samples>
                         <resolution>1</resolution>
-                        <min_angle>-1.0472</min_angle>
-                        <max_angle>0.0</max_angle>
+                        <min_angle>-0.2618</min_angle>
+                        <max_angle>0.2618</max_angle>
                     </vertical>
                 </scan>
+                <!-- Portée -->
                 <range>
                     <min>0.05</min>
@@ -224,10 +283,13 @@
         </sensor>
     </gazebo>
+    <!-- ================================================== -->
+    <!-- DIFF DRIVE                                         -->
+    <!-- ================================================== -->
     <gazebo>
         <plugin filename="gz-sim-diff-drive-system" name="gz::sim::systems::DiffDrive">
             <left_joint>left_wheel_joint</left_joint>
             <right_joint>right_wheel_joint</right_joint>
-            <wheel_separation>0.33</wheel_separation>
-            <wheel_radius>0.05</wheel_radius>
+            <wheel_separation>0.36</wheel_separation>
+            <wheel_radius>0.15</wheel_radius>
             <topic>/cmd_vel</topic>
             <odom_publish_frequency>30</odom_publish_frequency>
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